Commit message: modified joint limits

File: fanuc_r2000ic_support/urdf/r2000ic165f_macro.xacro (robot description, xacro)
@@ -115,5 +115,5 @@
       <child link="${prefix}link_1"/>
       <axis xyz="0 0 1"/>
-      <limit lower="${radians(-185)}" upper="${radians(185)}" effort="0" velocity="${radians(130)}"/>
+      <limit lower="${radians(-170)}" upper="${radians(170)}" effort="0" velocity="${radians(130)}"/>
     </joint>
     <joint name="${prefix}joint_2" type="revolute">
@@ -129,5 +129,5 @@
       <child link="${prefix}link_3"/>
       <axis xyz="0 -1 0"/>
-      <limit lower="${radians(-132)}" upper="${radians(180)}" effort="0" velocity="${radians(125)}"/>
+      <limit lower="${radians(-132)}" upper="${radians(230)}" effort="0" velocity="${radians(125)}"/>
     </joint>
     <joint name="${prefix}joint_4" type="revolute">
@@ -136,5 +136,5 @@
       <child link="${prefix}link_4"/>
       <axis xyz="-1 0 0"/>
-      <limit lower="${radians(-360)}" upper="${radians(360)}" effort="0" velocity="${radians(180)}"/>
+      <limit lower="${radians(-240)}" upper="${radians(240)}" effort="0" velocity="${radians(180)}"/>
     </joint>
     <joint name="${prefix}joint_5" type="revolute">
